File: bsc.kicad_pcb (KiCad board)
At the start: 4 copper layers, 120 x 100 mm, 288 parts, among them IC1 ILD217T, IC2 ILD217T, IC3 ILD217T, IC4 ILD217T, J1 Conn_JTAG_ESP, J10 JP_REL1_COM_12V, J12 JP_REL2_COM_12V, J13 JP_REL3_COM_12V, J14 Conn_REL1, J15 Conn_REL2, J16 Conn_REL3, J2 Prog, J3 Conn_Extension, J4 Boot, J5 JP_REL4_COM_12V, J6 JP_U3TX_EN, J8 JP_REL5_COM_12V, J9 JP_REL6_COM_12V, K2 TIANBO-HJR-4102-L, K3 TIANBO-HJR-4102-L, K4 TIANBO-HJR-4102-L, K5 TIANBO-HJR-4102-L, K6 TIANBO-HJR-4102-L, K7 TIANBO-HJR-4102-L, Q1 BC857BS, Q10 BC846, Q11 BC846, Q12 IRLML2244, Q13 BC857BS, Q14 IRLML2244, Q2 BSS138, Q3 BSS138, Q4 BSS138, Q5 BSS138, Q6 BSS138, Q7 BSS138, Q8 BC846, Q9 BC846, U1 LMO78_03-0.5, U10 74HC595, U11 74HC14, U12 74HC165, U13 ADuM1201AR, U14 NCP1117-3.3_SOT223, U15 NCP1117-3.3_SOT223, U16 SP3485EN, U17 NCP1117-3.3_SOT223, U19 LMO78_05-0.5, U2 ESP32WROOM32E16, U20 HC 151, U4 ADuM1201AR, U5 ADuM1201AR, U6 ADuM1201AR, U7 SN65HVD234, U8 SP3485EN, U9 SP3485EN, X1 Conn_S2, X2 Conn_S1, X3 Conn_DI, X4 Conn_SV, X5 Conn_Rel2, X6 Conn_Rel1

Commit message: Ref 2.4
Parts:
- removed C36, C37, C45: 100n, Capacitor_SMD:C_0603_1608Metric
- removed D2, D24, D3: LL4148, Diode_SMD:D_MiniMELF
- removed IC4: ILD217T, Package_SO:SOIC-8_3.9x4.9mm_P1.27mm
- removed JP25: JP_U3_RXS_RXO, Jumper:SolderJumper-2_P1.3mm_Open_RoundedPad1.0x1.5mm
- removed JP26: JP_U3_TXS_TXO, Jumper:SolderJumper-2_P1.3mm_Open_RoundedPad1.0x1.5mm
- removed JP27: JP_U3_TXEN_TXENS, Jumper:SolderJumper-2_P1.3mm_Open_RoundedPad1.0x1.5mm
- removed R61, R87: 2k2, Resistor_SMD:R_0603_1608Metric
- removed R86: 330R, Resistor_SMD:R_0603_1608Metric
- removed U14, U15, U17: NCP1117-3.3_SOT223, Package_TO_SOT_SMD:SOT-223-3_TabPin2
- removed U5: ADuM1201AR, Package_SO:SOIC-8_3.9x4.9mm_P1.27mm
- removed U9: SP3485EN, Package_SO:SOIC-8_3.9x4.9mm_P1.27mm
- added JP32: JP_U1_120R, Jumper:SolderJumper-2_P1.3mm_Open_RoundedPad1.0x1.5mm, B.Cu at (65.3, 40.8)
- added JP33: JP_U2_120R, Jumper:SolderJumper-2_P1.3mm_Open_RoundedPad1.0x1.5mm, B.Cu at (74.9, 40.8)
- added JP34: JP_U3_120R, Jumper:SolderJumper-2_P1.3mm_Open_RoundedPad1.0x1.5mm, B.Cu at (96.2, 36.4)
- added R88: 120R, Resistor_SMD:R_0603_1608Metric, B.Cu at (68.5, 40.3)
- added R89: 120R, Resistor_SMD:R_0603_1608Metric, B.Cu at (77.3, 40.9)
- added R90: 120R, Resistor_SMD:R_0603_1608Metric, B.Cu at (96.3, 34.3)
- added RJ1: R-RJ45S08P-B000, lcsc:RJ45-TH_R-RJ45S08P-B000, F.Cu at (103.3, 39.4)
- added U3: ADM2483xRW, Package_SO:SOIC-16W_7.5x10.3mm_P1.27mm, B.Cu at (97.5, 58.4)
- C31, C33, C35, C38, C39, C42: moved to B.Cu
- JP28, JP30, JP31: footprint Jumper:SolderJumper-2_P1.3mm_Open_RoundedPad1.0x1.5mm -> Jumper:SolderJumper-2_P1.3mm_Bridged_RoundedPad1.0x1.5mm
- JP29: footprint Jumper:SolderJumper-3_P1.3mm_Open_RoundedPad1.0x1.5mm -> Jumper:SolderJumper-3_P1.3mm_Bridged12_RoundedPad1.0x1.5mm_NumberLabels
- PS1, PS3, PS4, PS5: value 1S4E_0503S1U -> B0503S-1WR2; footprint custom_th:Converter_DCDC_GAPTEC_1S4E_S1U -> lcsc:PWRM-TH_DEXU_BXXXXS-1WR2
- PS2: value 1S4E_0505S1U -> B0505S-1WR2_C909796; footprint custom_th:Converter_DCDC_GAPTEC_1S4E_S1U -> lcsc:PWRM-TH_BXXXXS-1WR3
- R59: value 330R -> 10k
- X1: footprint Connector_Phoenix_MC:PhoenixContact_MCV_1,5_9-G-3.81_1x09_P3.81mm_Vertical -> Connector_Phoenix_MC:PhoenixContact_MCV_1,5_6-G-3.81_1x06_P3.81mm_Vertical
- moved C43 15.9 mm to (102.9, 64.8), turned to 0 degrees
- moved X1 15.7 mm to (35.1, 37.0)
- moved JP23 14.3 mm to (98.8, 48.3)
- moved X2 14.2 mm to (76.1, 37.0)
- moved JP24 11.0 mm to (95.5, 51.8), turned to 0 degrees
- moved C42 9.50 mm to (87.8, 44.3)
- moved R59 8.42 mm to (93.0, 57.9), turned to -90 degrees
- moved C47 6.85 mm to (93.2, 64.8), turned to 180 degrees
- moved C35 6.17 mm to (103.9, 46.7), turned to 0 degrees
- moved C33 6.13 mm to (103.6, 48.9), turned to 0 degrees
- moved JP16 5.77 mm to (89.1, 56.6), turned to 180 degrees
- moved C39 5.11 mm to (89.8, 44.2)
- moved R64 4.01 mm to (103.2, 44.5), turned to 180 degrees
- moved JP22 4.01 mm to (105.5, 53.8)
- moved PS1 3.88 mm to (67.6, 47.0), turned to 90 degrees
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Connections:
- C13 pad 1: +5V -> GND
- C13 pad 2: GND -> +5V
- C32 pad 2: /U1_GND -> /serial/U1_GND
- C34 pad 2: /U1_GND -> /serial/U1_GND
- C40 pad 2: /U1_GND -> /serial/U1_GND
- JP11 pad 2: /U1RX_O -> /serial/U1RX_O
- JP12 pad 2: /U1TX_O -> /serial/U1TX_O
- JP23 pad 2: /serial/U3RX_S -> /serial/U3RX_O
- JP24 pad 2: /serial/U3TX_S -> /serial/U3TX_O
- JP28 pad 1: V_IN -> +5V
- JP28 pad 2: +5V -> V_IN
- JP8 pad 2: /U1_GND -> /serial/U1_GND
- PS3 pad 3: /U1_GND -> /serial/U1_GND
- R59 pad 2: /U3RXTX_EN -> +3V3
- R60 pad 2: /U1_GND -> /serial/U1_GND
- R63 pad 1: /U1_GND -> /serial/U1_GND
- U4 pad 5: /U1_GND -> /serial/U1_GND
- U8 pad 5: /U1_GND -> /serial/U1_GND
- U8 pad 6: /U1RX_O -> /serial/U1RX_O
- U8 pad 7: /U1TX_O -> /serial/U1TX_O
- X1 pad 6: /U1_VCC_e -> /CAN_GND
- X2 pad 1: /serial/U2_VCC_e -> /serial/U1_GND
- X2 pad 2: /serial/U2_GND -> /serial/U1TX_O
- X2 pad 3: /serial/U2TX_O -> /serial/U1RX_O
- X2 pad 4: /serial/U2RX_O -> /serial/U2_GND
- X2 pad 5: /serial/U3_VCC_e -> /serial/U2TX_O
- X2 pad 6: /serial/U3_GND -> /serial/U2RX_O
- X2 pad 7: /serial/U3TX_O -> /serial/U3_GND
- X2 pad 8: /serial/U3RX_O -> /serial/U3TX_O
- X2 pad 9: GND -> /serial/U3RX_O
Routing:
- net /U1_GND: track 44.7 -> 0.00 mm, vias 4 -> 0
- net /serial/U3_GND: track 38.0 -> 80.9 mm, vias 6 -> 0
- net /serial/U1_GND: track 0.00 -> 36.9 mm, vias 0 -> 4
- net /serial/U1RX_O: track 0.00 -> 32.2 mm
- net /serial/U3TX_O: track 29.0 -> 58.9 mm
- net /U1RX_O: track 29.7 -> 0.00 mm
- net /U1TX_O: track 27.4 -> 0.00 mm, vias 3 -> 0
- net /serial/U1TX_O: track 0.00 -> 26.7 mm, vias 0 -> 2
- net /serial/U3_VCC: track 42.3 -> 18.7 mm, vias 4 -> 1
- net Net-(C45-Pad1): track 22.8 -> 0.00 mm, vias 2 -> 0
- net /serial/U3RX_O: track 24.7 -> 45.9 mm, vias 2 -> 0
- net /serial/U3RXTX_ENs: track 20.9 -> 0.00 mm, vias 1 -> 0
- net Net-(C36-Pad1): track 18.8 -> 0.00 mm
- net GND: track 383.0 -> 364.3 mm, vias 73 -> 71
- net /U3RX: track 91.5 -> 104.3 mm, vias 1 -> 3
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- added copper zone on In1.Cu, net /serial/U1_GND
- removed copper zone on In1.Cu, net /U1_GND
Other:
- board text added: "1: Analogeingang 2: +5/+12V OUT (je nach Bestück.) 3: +5V OUT 4: +3V3 OUT 5: GND 6: GND"
- board text added: "1: GND 2: +3V3 3: Onewire"
- board text added: "1: Rel 1 (NO) 2: Rel 1 (COM) 3: Rel 1 (NC)/Tacho 1 4: Rel 2 (NO) 5: Rel 2 (COM) 6: Rel 2 (NC)/Tacho 2"
- board text added: "1: Rel 4 (NO) 2: Rel 4 (COM) 3: Tacho 4 4: Rel 5 (NO) 5: Rel 5 (COM) 6: Tacho 5"
- board text added: "1: S0 GND 2: S0 TX/B 3: S0 RX/A"
- board text added: "4: CAN_H 5: CAN_L 6: CAN_GND"
- board text added: "4: S1 GND 5: S1 TX/B 6: S1 RX/A"
- board text added: "7: GND 8: V IN2 9: V IN1"
- board text added: "7: Rel 3 (NO) 8: Rel 3 (COM) 9: Rel 2 (NC)/Tacho 3"
- board text added: "7: Rel 6 (NO) 8: Rel 6 (COM) 9: Tacho 6"
- board text added: "7: S2 GND 8: S2 TX/B 9: S2 RX/A"
- board text added: "PCB V2.4"
- board text added: "U1|U2|U3| JP 07|14|21|3V3->Ux_VCC JP 08|15|22|GND->Ux_GND JP 09|16|23|UxRX->UxRX_S JP 10|17|24|UxTX->UxTX_S JP 11|18|- |UxRX_S->UxRX_O JP 12|19|- |UxTX_S->UxTX_O JP 13|20|- |UxRXTX_EN->UxRXTX_ENs"
- board text removed: "1: Analogeingang 2: +5/+12V OUT (je nach Bestück.) 3: +5V OUT 4: +3V3 OUT"
- board text removed: "1: GND 2: +3V3 3: Onewire 4: CAN H 5: CAN L"
- board text removed: "1: Rel 1 (NO) 2: Rel 1 (COM) 3: Rel 1 (NC)/Tacho 1"
- board text removed: "1: Rel 4 (NO) 2: Rel 4 (COM) 3: Tacho 4"
- board text removed: "1: U2 VCC 2: U2 GND 3: U2 TX 4: U2 RX"
- board text removed: "4: Rel 2 (NO) 5: Rel 2 (COM) 6: Rel 2 (NC)/Tacho 2 7: Rel 3 (NO) 8: Rel 3 (COM) 9: Rel 2 (NC)/Tacho 3"
- board text removed: "4: Rel 5 (NO) 5: Rel 5 (COM) 6: Tacho 5 7: Rel 6 (NO) 8: Rel 6 (COM) 9: Tacho 6"
- board text removed: "5: GND 6: GND 7: GND 8: V IN2 9: V IN1"
- board text removed: "5: U3 VCC 6: U3 GND 7: U3 TX 8: U3 RX 9: GND"
- board text removed: "6: U1 VCC 7: U1 GND 8: U1 TX 9: U1 RX"
- board text removed: "Battery safety controller V2.3 github.com/shining-man/bsc_fw created by shiningman"
- board text removed: "U1|U2|U3| JP 07|14|21|3V3->Ux_VCC JP 08|15|22|GND->Ux_GND JP 09|16|23|UxRX->UxRX_S JP 10|17|24|UxTX->UxTX_S JP 11|18|25|UxRX_S->UxRX_O JP 12|19|26|UxTX_S->UxTX_O JP 13|20|27|UxRXTX_EN->UxRXTX_ENs"
