File: bsc.kicad_pcb (KiCad board)
At the start: 4 copper layers, 120 x 100 mm, 286 parts, among them IC1 ILD217T, IC2 ILD217T, IC3 ILD217T, J1 Conn_JTAG_ESP, J10 JP_REL1_COM_12V, J12 JP_REL2_COM_12V, J13 JP_REL3_COM_12V, J14 Conn_REL1, J15 Conn_REL2, J16 Conn_REL3, J2 Prog, J3 Conn_Extension, J4 Boot, J5 JP_REL4_COM_12V, J6 JP_U3TX_EN, J8 JP_REL5_COM_12V, J9 JP_REL6_COM_12V, K2 TIANBO-HJR-4102-L, K3 TIANBO-HJR-4102-L, K4 TIANBO-HJR-4102-L, K5 TIANBO-HJR-4102-L, K6 TIANBO-HJR-4102-L, K7 TIANBO-HJR-4102-L, Q1 BC857BS, Q10 BC846, Q11 BC846, Q12 IRLML2244, Q13 BC857BS, Q14 IRLML2244, Q15 BSS138, Q2 BSS138, Q3 BSS138, Q4 BSS138, Q5 BSS138, Q6 BSS138, Q7 BSS138, Q8 BC846, Q9 BC846, U1 K7803-1000R3, U10 74HC595, U11 74HC14, U12 74HC165, U13 ADuM1201AR, U16 SP3485EN, U19 LMO78_05-0.5, U2 ESP32WROOM32E16, U20 HC 151, U3 ADM2483xRW, U4 ADuM1201AR, U6 ADuM1201AR, U7 SN65HVD234, U8 SP3485EN, X1 Conn_S2, X2 Conn_S1, X3 Conn_DI, X4 Conn_SV, X5 Conn_Rel2, X6 Conn_Rel1

Commit message: Version geändert
Other:
- board text added: "PCB V2.5 https://github.com/shining-man/bsc_hw"
- board text removed: "PCB V2.4.1 https://github.com/shining-man/bsc_hw"
Changed lines of the file:
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@@
     (effects (font (size 1 1) (thickness 0.15)) (justify left mirror))
   )
-  (gr_text "PCB V2.4.1\nhttps://github.com/shining-man/bsc_hw" (at 34.1884 72.39 270) (layer "B.SilkS")
+  (gr_text "PCB V2.5\nhttps://github.com/shining-man/bsc_hw" (at 34.1884 72.39 270) (layer "B.SilkS")
     (effects (font (size 1.1 1.1) (thickness 0.15)) (justify left mirror))
   )

Commit message: Layoutänderungen
Routing:
- net GND: track 368.7 -> 360.3 mm, vias 71 -> 69
- net +3V3: vias 33 -> 32
