File: bsc.kicad_sch (KiCad schematic)
At the start: 74 parts, among them J1 Conn_JTAG_ESP, J2 Prog, J3 Conn_Extension, J4 Boot, J6 JP_U3TX_EN, Q1 BC857BS, Q12 IRLML2244, Q13 BC857BS, Q14 IRLML2244, U1 K7803-1000R3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

Commit message: Layoutänderungen
Parts:
- J1, U19: now left out of the parts list
Changed lines of the file:
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@@
   (title_block
     (title "BSC")
-    (date "2024-04-07")
+    (date "2024-04-16")
     (rev "2.5")
   )
@@
   )
   (symbol (lib_id "Connector_Generic:Conn_02x10_Odd_Even") (at 128.905 31.75 0) (unit 1)
-    (in_bom yes) (on_board yes) (dnp yes) (fields_autoplaced)
+    (in_bom no) (on_board yes) (dnp yes) (fields_autoplaced)
     (property "Reference" "J1" (at 130.175 16.6202 0)
       (effects (font (size 1.27 1.27)))
@@
   )
   (symbol (lib_id "Regulator_Switching:R-78E3.3-0.5") (at 135.255 154.305 0) (unit 1)
-    (in_bom yes) (on_board yes) (dnp yes) (fields_autoplaced)
+    (in_bom no) (on_board yes) (dnp yes) (fields_autoplaced)
     (property "Reference" "U19" (at 135.255 148.7002 0)
       (effects (font (size 1.27 1.27)))
